Commit message: Added support for parsing spherical joint

File: examples/01-robot_parse/pbot.urdf (robot description, URDF)
Before this commit: robot PBot, 2 links, 1 joints
Links:
- added link link1, mass 1
Joints:
- added joint sj1: type spherical, parent link0, child link1, origin xyz=0.000000 0.000000 3.000000 rpy=-0.000000 0.000000 -0.000000
